Commit message: configures metrics

File: hector_quadrotor/hector_quadrotor_description/urdf/quadrotor_hokuyo_utm30lx.urdf.xacro (robot description, xacro)
@@ -9,5 +9,5 @@
     <xacro:include filename="$(find hector_sensors_description)/urdf/hokuyo_utm30lx.urdf.xacro" />
     <xacro:hokuyo_utm30lx name="laser0" parent="base_link" ros_topic="scan" update_rate="40" ray_count="1081" min_angle="-135" max_angle="135">
-      <origin xyz="0.0 0.0 -0.097" rpy=" 0 1.54  0"/>
+      <origin xyz="0.0 0.0 -0.097" rpy=" 0 0  0"/>
     </xacro:hokuyo_utm30lx>
     <!-- Forward facing camera -->

File: husky/ugv_description/urdf/description.gazebo.xacro (robot description, xacro)
@@ -52,4 +52,23 @@
 		</collision>
 	</link>
+          <link name="laser_link1">
+		<inertial>
+			<mass value="1e-5" />
+			<origin xyz="0 0 0" rpy="0 0 0" />
+			<inertia ixx="1e-6" ixy="0" ixz="0" iyy="1e-6" iyz="0" izz="1e-6" />
+		</inertial>
+		<visual>
+			<origin xyz="0 0 0" rpy="0 0 0" />
+			<geometry>
+				<box size="0.01 0.01 0.01" />
+			</geometry>
+		</visual>
+		<collision>
+			<origin xyz="0 0 0" rpy="0 0 0" />
+			<geometry>
+				<box size="0.01 0.01 0.01" />
+			</geometry>
+		</collision>
+	</link>
 	<joint name="laser_joint" type="fixed">
 		<axis xyz="0 1 0" />
@@ -57,4 +76,10 @@
 		<parent link="base_link" />
 		<child link="laser_link" />
+	</joint>
+        	<joint name="laser_joint1" type="fixed">
+		<axis xyz="0 1 0" />
+		<origin xyz="1 0 0.3" rpy="0 0 0" />
+		<parent link="base_link" />
+		<child link="laser_link1" />
 	</joint>
 	<!-- GPS -->

File: husky/ugv_description/urdf/husky.gazebo.xacro (robot description, xacro)
@@ -92,4 +92,41 @@
 	  </sensor>
 	  </gazebo>
+   <gazebo reference="laser_link1">
+	  <sensor name="sensor" type="ray">
+	    <always_on>true</always_on>
+	    <update_rate>5</update_rate>
+	    <visualize>false</visualize>
+	    <ray>
+	      <scan>
+		<horizontal>
+		  <samples>720</samples>
+		  <resolution>1</resolution>
+		  <min_angle>-3.14</min_angle> <!--135 derece -> 2.35619 radyan-->
+		  <max_angle>3.14</max_angle>  <!--135 derece -> 2.35619 radyan-->
+		</horizontal>
+		<vertical>
+		  <samples>16</samples> <!--lazer katman sayisi-->
+		  <resolution>1</resolution>
+		  <min_angle>-0.20</min_angle> <!--radyan-->
+		  <max_angle>0.261</max_angle> <!--radyan-->
+		</vertical>
+	      </scan>
+	      <range>
+		<min>0.65</min> <!--metre-->
+		<max>50</max> <!--metre-->
+		<resolution>0.02</resolution>
+	      </range>
+	    </ray>
+	    <plugin name="gazebo_ros_laser_controller_1" filename="libgazebo_ros_velodyne_laser.so"> <!-- https://bitbucket.org/DataspeedInc/velodyne_simulator.git -->
+	      <frameName>laser_link</frameName>
+	      <topicName>ugv/cloud1</topicName>
+	      <gaussianNoise>0.02</gaussianNoise>
+	      <hokuyoMinIntensity>1</hokuyoMinIntensity>
+	      <alwaysOn>true</alwaysOn>
+	      <updateRate>5</updateRate>
+	      <pcl>2.0</pcl>
+	    </plugin>
+	  </sensor>
+	  </gazebo>
   </xacro:macro>
 </robot>
